Commit message: second commit

File: src/mybot_description/urdf/mybot.xacro (robot description, xacro)
@@ -165,6 +165,6 @@
   </joint>
   <joint name="hokuyo_joint" type="fixed">
-    <axis xyz="0 1 0" />
-    <origin xyz=".15 0 .1" rpy="0 0 0"/>
+    <axis xyz="0 1 0.1" />
+    <origin xyz=".15 0 .15" rpy="0 0 0"/>
     <parent link="chassis"/>
     <child link="hokuyo"/>
